File: kiCad/OLED_Display.kicad_sch (KiCad schematic)
At the start: 1 part, among them U4 OLED_DISPLAY_SSD1306_SPI

Commit message: Lots of stuff
Parts:
- U4: footprint (none) -> CustomFootprints:HiLetgo_OLED_SPI
Changed lines of the file:
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@@
 			)
 		)
-		(property "Footprint" ""
+		(property "Footprint" "CustomFootprints:HiLetgo_OLED_SPI"
 			(at 139.7 93.98 0)
 			(effects
@@
 					(size 1.27 1.27)
 				)
-				(hide yes)
 			)
 		)
